File: schem/toastflow.sch (KiCad schematic (older format))
At the start: 21 parts, among them IC1 ATTINY13, K1 CONN_3, P1 CONN_3X2, SW1 SW_PUSH, U1 TRIAC

Commit message: Fixed triac pin.
Connections:
- net TRIAC: now reaches IC1.7 (PB2(SCK/ADC1/T0/PCINT2)), P1.3
- net TRIAC: now also R3.2
Changed lines of the file:
@@
-EESchema Schematic File Version 2  date E 18 veebr 2013 16:26:19 EET
+EESchema Schematic File Version 2  date K 20 veebr 2013 23:50:52 EET
 LIBS:tech-thing
 LIBS:toastflow-cache
@@
 Sheet 1 1
 Title ""
-Date "18 feb 2013"
+Date "20 feb 2013"
 Rev ""
 Comp ""
@@
 F 0 "U1" H 3100 3300 70  0000 C CNN
 F 1 "TRIAC" H 3050 2700 60  0000 C CNN
+F 2 "" H 3350 2950 60  0001 C CNN
+F 3 "" H 3350 2950 60  0001 C CNN
 	1    3350 2950
 	-1   0    0    1
@@
 F 0 "K1" V 2450 3250 50  0000 C CNN
 F 1 "CONN_3" V 2550 3250 40  0000 C CNN
+F 2 "" H 2500 3250 60  0001 C CNN
+F 3 "" H 2500 3250 60  0001 C CNN
 	1    2500 3250
 	-1   0    0    1
@@
 F 0 "F1" H 3200 2750 40  0000 C CNN
 F 1 "FUSE" H 3000 2650 40  0000 C CNN
+F 2 "" H 3100 2700 60  0001 C CNN
+F 3 "" H 3100 2700 60  0001 C CNN
 	1    3100 2700
 	1    0    0    -1
@@
 F 1 "ATTINY13" H 7100 3800 60  0000 C CNN
 F 2 "DIP8" H 5900 3800 60  0001 C CNN
+F 3 "" H 5800 4550 60  0001 C CNN
 	1    5800 4550
 	1    0    0    -1
@@
 F 0 "#PWR01" H 7600 4750 30  0001 C CNN
 F 1 "VCC" H 7600 4750 30  0000 C CNN
+F 2 "" H 7600 4650 60  0001 C CNN
+F 3 "" H 7600 4650 60  0001 C CNN
 	1    7600 4650
 	1    0    0    -1
@@
 F 0 "#PWR02" H 7600 5150 30  0001 C CNN
 F 1 "GND" H 7600 5080 30  0001 C CNN
+F 2 "" H 7600 5150 60  0001 C CNN
+F 3 "" H 7600 5150 60  0001 C CNN
 	1    7600 5150
 	1    0    0    -1
@@
 F 0 "C4" H 7650 5000 50  0000 L CNN
 F 1 "100n" H 7650 4800 50  0000 L CNN
+F 2 "" H 7600 4900 60  0001 C CNN
+F 3 "" H 7600 4900 60  0001 C CNN
 	1    7600 4900
 	1    0    0    -1
@@
 F 0 "R3" V 4180 2750 50  0000 C CNN
 F 1 "47" V 4100 2750 50  0000 C CNN
+F 2 "" H 4100 2750 60  0001 C CNN
+F 3 "" H 4100 2750 60  0001 C CNN
 	1    4100 2750
 	0    -1   -1   0
@@
 F 0 "P1" H 4750 5150 50  0000 C CNN
 F 1 "CONN_3X2" V 4750 4950 40  0000 C CNN
+F 2 "" H 4750 4900 60  0001 C CNN
+F 3 "" H 4750 4900 60  0001 C CNN
 	1    4750 4900
 	-1   0    0    -1
@@
 F 0 "#PWR03" H 4350 4850 30  0001 C CNN
 F 1 "VCC" H 4350 4850 30  0000 C CNN
+F 2 "" H 4350 4750 60  0001 C CNN
+F 3 "" H 4350 4750 60  0001 C CNN
 	1    4350 4750
 	-1   0    0    -1
@@
 F 0 "#PWR04" H 4350 4950 30  0001 C CNN
 F 1 "GND" H 4350 4880 30  0001 C CNN
+F 2 "" H 4350 4950 60  0001 C CNN
+F 3 "" H 4350 4950 60  0001 C CNN
 	1    4350 4950
 	-1   0    0    -1
@@
 F 0 "R5" V 4980 5150 50  0000 C CNN
 F 1 "100k" V 4900 5150 50  0000 C CNN
+F 2 "" H 4900 5150 60  0001 C CNN
+F 3 "" H 4900 5150 60  0001 C CNN
 	1    4900 5150
 	0    -1   -1   0
@@
 F 0 "#PWR05" H 4650 5250 30  0001 C CNN
 F 1 "VCC" H 4650 5250 30  0000 C CNN
+F 2 "" H 4650 5150 60  0001 C CNN
+F 3 "" H 4650 5150 60  0001 C CNN
 	1    4650 5150
 	1    0    0    -1
@@
 F 0 "D3" H 6250 3600 50  0000 C CNN
 F 1 "LED" H 6250 3400 50  0000 C CNN
+F 2 "" H 6250 3500 60  0001 C CNN
+F 3 "" H 6250 3500 60  0001 C CNN
 	1    6250 3500
 	1    0    0    -1
@@
 F 0 "R6" V 5880 3500 50  0000 C CNN
 F 1 "1k" V 5800 3500 50  0000 C CNN
+F 2 "" H 5800 3500 60  0001 C CNN
+F 3 "" H 5800 3500 60  0001 C CNN
 	1    5800 3500
 	0    -1   -1   0
@@
 F 0 "#PWR06" H 6450 3500 30  0001 C CNN
 F 1 "GND" H 6450 3430 30  0001 C CNN
+F 2 "" H 6450 3500 60  0001 C CNN
+F 3 "" H 6450 3500 60  0001 C CNN
 	1    6450 3500
 	1    0    0    -1
@@
 F 0 "SW1" H 5150 3910 50  0000 C CNN
 F 1 "SW_PUSH" H 5000 3720 50  0000 C CNN
+F 2 "" H 5000 3800 60  0001 C CNN
+F 3 "" H 5000 3800 60  0001 C CNN
 	1    5000 3800
 	0    1    1    0
@@
 F 0 "C3" H 4800 3900 50  0000 L CNN
 F 1 "C" H 4800 3700 50  0000 L CNN
+F 2 "" H 4750 3800 60  0001 C CNN
+F 3 "" H 4750 3800 60  0001 C CNN
 	1    4750 3800
 	-1   0    0    -1
@@
 F 0 "#PWR07" H 4750 4100 30  0001 C CNN
 F 1 "GND" H 4750 4030 30  0001 C CNN
+F 2 "" H 4750 4100 60  0001 C CNN
+F 3 "" H 4750 4100 60  0001 C CNN
 	1    4750 4100
 	1    0    0    -1
@@
 F 0 "R4" V 4830 3250 50  0000 C CNN
 F 1 "100k" V 4750 3250 50  0000 C CNN
+F 2 "" H 4750 3250 60  0001 C CNN
+F 3 "" H 4750 3250 60  0001 C CNN
 	1    4750 3250
 	1    0    0    -1
@@
 F 0 "#PWR08" H 4750 3100 30  0001 C CNN
 F 1 "VCC" H 4750 3100 30  0000 C CNN
+F 2 "" H 4750 3000 60  0001 C CNN
+F 3 "" H 4750 3000 60  0001 C CNN
 	1    4750 3000
 	1    0    0    -1
@@
 F 0 "TH1" V 7700 3350 50  0000 C CNN
 F 1 "THERMISTOR" V 7500 3300 50  0000 C CNN
+F 2 "" H 7600 3300 60  0001 C CNN
+F 3 "" H 7600 3300 60  0001 C CNN
 	1    7600 3300
 	1    0    0    -1
@@
 F 0 "#PWR09" H 7600 3150 30  0001 C CNN
 F 1 "VCC" H 7600 3150 30  0000 C CNN
+F 2 "" H 7600 3050 60  0001 C CNN
+F 3 "" H 7600 3050 60  0001 C CNN
 	1    7600 3050
 	1    0    0    -1
@@
 F 0 "R7" V 7680 3800 50  0000 C CNN
 F 1 "100k" V 7600 3800 50  0000 C CNN
+F 2 "" H 7600 3800 60  0001 C CNN
+F 3 "" H 7600 3800 60  0001 C CNN
 	1    7600 3800
 	1    0    0    -1
@@
 F 0 "#PWR010" H 7600 4050 30  0001 C CNN
 F 1 "GND" H 7600 3980 30  0001 C CNN
+F 2 "" H 7600 4050 60  0001 C CNN
+F 3 "" H 7600 4050 60  0001 C CNN
 	1    7600 4050
 	1    0    0    -1
@@
 F 0 "R1" V 2830 4800 50  0000 C CNN
 F 1 "47" V 2750 4800 50  0000 C CNN
+F 2 "" H 2750 4800 60  0001 C CNN
+F 3 "" H 2750 4800 60  0001 C CNN
 	1    2750 4800
 	0    -1   -1   0
@@
 F 0 "C1" H 2350 4900 50  0000 L CNN
 F 1 "100n" H 2350 4700 50  0000 L CNN
+F 2 "" H 2300 4800 60  0001 C CNN
+F 3 "" H 2300 4800 60  0001 C CNN
 	1    2300 4800
 	0    -1   -1   0
@@
 F 0 "C2" H 3450 4700 50  0000 L CNN
 F 1 "100u" H 3450 4500 50  0000 L CNN
+F 2 "" H 3400 4600 60  0001 C CNN
+F 3 "" H 3400 4600 60  0001 C CNN
 	1    3400 4600
 	1    0    0    -1
@@
 F 0 "#PWR011" H 3400 4800 30  0001 C CNN
 F 1 "GND" H 3400 4730 30  0001 C CNN
+F 2 "" H 3400 4800 60  0001 C CNN
+F 3 "" H 3400 4800 60  0001 C CNN
 	1    3400 4800
 	1    0    0    -1
@@
 F 0 "#PWR012" H 3400 4500 30  0001 C CNN
 F 1 "VCC" H 3400 4500 30  0000 C CNN
+F 2 "" H 3400 4400 60  0001 C CNN
+F 3 "" H 3400 4400 60  0001 C CNN
 	1    3400 4400
 	1    0    0    -1
@@
 F 0 "R2" V 3280 3700 50  0000 C CNN
 F 1 "1M" V 3200 3700 50  0000 C CNN
+F 2 "" H 3200 3700 60  0001 C CNN
+F 3 "" H 3200 3700 60  0001 C CNN
 	1    3200 3700
 	0    -1   -1   0
@@
 F 0 "D2" H 3200 4900 40  0000 C CNN
 F 1 "DIODE" H 3200 4700 40  0000 C CNN
+F 2 "" H 3200 4800 60  0001 C CNN
+F 3 "" H 3200 4800 60  0001 C CNN
 	1    3200 4800
 	1    0    0    -1
@@
 F 0 "D1" H 3000 4650 40  0000 C CNN
 F 1 "ZENER" H 3000 4450 30  0000 C CNN
+F 2 "" H 3000 4550 60  0001 C CNN
+F 3 "" H 3000 4550 60  0001 C CNN
 	1    3000 4550
 	0    1    1    0
@@
 F 0 "#PWR013" H 3350 2800 30  0001 C CNN
 F 1 "VCC" H 3350 2800 30  0000 C CNN
+F 2 "" H 3350 2700 60  0001 C CNN
+F 3 "" H 3350 2700 60  0001 C CNN
 	1    3350 2700
 	1    0    0    -1
@@
 Text Label 3450 3700 0    60   ~ 0
 SENSE
+Text Label 4350 2750 0    60   ~ 0
+TRIAC
+Text Label 5600 4850 2    60   ~ 0
+TRIAC
+Connection ~ 5600 4850
 $EndSCHEMATC

Commit message: Component fix
Parts:
- R7: value 100k -> 2k2
Changed lines of the file:
@@
-EESchema Schematic File Version 2  date K 20 veebr 2013 23:50:52 EET
+EESchema Schematic File Version 2  date K 27 veebr 2013 22:57:51 EET
 LIBS:tech-thing
 LIBS:toastflow-cache
@@
 Sheet 1 1
 Title ""
-Date "20 feb 2013"
+Date "27 feb 2013"
 Rev ""
 Comp ""
@@
 P 7600 3800
 F 0 "R7" V 7680 3800 50  0000 C CNN
-F 1 "100k" V 7600 3800 50  0000 C CNN
+F 1 "2k2" V 7600 3800 50  0000 C CNN
 F 2 "" H 7600 3800 60  0001 C CNN
 F 3 "" H 7600 3800 60  0001 C CNN
